File: Hardware/MorseCode/MorseCode.kicad_sch (KiCad schematic)
At the start: 7 parts

Commit message: Initial MorseCode Hardware prototype
Parts:
- renumbered Z to Z1
Changed lines of the file:
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@@
 		(dnp no)
 		(fields_autoplaced yes)
-		(property "Reference" "Z"
+		(property "Reference" "Z1"
 			(at 254 38.1 0)
 			(hide yes)
@@
 			(project "MorseCode"
 				(path "/16bba23a-a500-415f-8344-fab3afafd4a7"
-					(reference "Z")
+					(reference "Z1")
 					(unit 1)
 				)
