File: Hardware/CanBusModule/CanBusModule.kicad_sch (KiCad schematic)
At the start: 17 parts, among them U1 XIAO-ESP32-S3-Plus-SMD, U2 MCP2518FDT-E_QBB, U3 ATA6561-GBQW-N, U4 74HCT1G125GW, Y1 ECS-400-15-33B-CTN-TR

Commit message: Commiting an interim commit before chatgpt breaks it more
Connections:
- net at U3.8 (STBY): now also U2.9 (~{INT0}/GPIO0/XSTBY)
Changed lines of the file:
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@@
+	(wire
+		(pts
+			(xy 196.215 97.79) (xy 191.77 97.79)
+		)
+		(stroke
+			(width 0)
+			(type default)
+		)
+	)
 	(wire
 		(pts
@@
 	(wire
 		(pts
+			(xy 196.215 123.19) (xy 196.215 97.79)
+		)
+		(stroke
+			(width 0)
+			(type default)
+		)
+	)
+	(wire
+		(pts
 			(xy 185.42 38.735) (xy 185.42 43.815)
 		)
 		(stroke
+			(width 0)
+			(type default)
+		)
+	)
+	(wire
+		(pts
+			(xy 182.88 123.19) (xy 196.215 123.19)
+		)
+		(stroke
